File: Hardware/E-book_Reader.brd (EAGLE design)
At the start: 170.2 x 111.2 mm, 103 parts, among them IC1 BD5229G-TR, IC4 XC6220A331MR-G, J1 FH34SRJ-24S-0.5SH_99_, J2 SAMACSYS_PARTS_USB4110-GF-A, J3 QWIIC_RIGHT_ANGLE, J4 112A-TAAR-R03_ATTEND, Q1 20V/4.2A/52mΩ/1.4W, Q2 20V/4.2A/52mΩ/1.4W, Q3 SI1308EDL-T1-GE3, U1 W25Q512JVEIQ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

Commit message: Add files via upload
Parts:
- removed R2_PINH5: 10k, DeskAssistant v19 v1:ESP32_WROVER_EAGLE-LTSPICE_R0402
- added R1: 10k, DeskAssistant v19 v1:ESP32_WROVER_EAGLE-LTSPICE_R0402
- moved TP16 53.4 mm to (65.9, 30.4)
- moved TP17 53.3 mm to (66.1, 24.1)
- moved TP14 49.3 mm to (18.0, 67.2)
- moved TP12 49.1 mm to (8.24, 67.3)
- moved TP15 44.1 mm to (22.5, 67.2)
- moved TP13 43.6 mm to (13.2, 67.2)
- moved R5 38.5 mm to (57.6, 47.8), turned to 0 degrees
- moved TP11 26.8 mm to (27.4, 38.2)
- moved TP4 20.2 mm to (23.4, 42.2)
- moved TP5 16.6 mm to (27.1, 42.3)
- moved TP2 15.8 mm to (11.0, 42.4)
- moved TP6 12.0 mm to (6.94, 38.4)
- moved TP3 11.1 mm to (15.0, 42.4)
- moved TP8 9.96 mm to (14.9, 38.2)
- moved TP1 9.75 mm to (6.94, 42.5)
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Connections:
- net 3V3: now also R1.1, R5.2; no longer R2_PINH5.2, R5.1
- net FLASH_CS: now also R5.1; no longer R2_PINH5.1
- net GPIO8: now also R1.2; no longer R5.2
Routing:
- net EPD_3V3: track 145.0 -> 86.6 mm
- net EPD_3V3_C: track 117.4 -> 66.3 mm, vias 2 -> 0
- net 3V3: track 449.9 -> 417.4 mm, vias 7 -> 6
- net EPD_CS: track 156.7 -> 126.0 mm, vias 5 -> 6
- net EPD_RST: track 142.3 -> 117.6 mm, vias 6 -> 2
- net 32KHZ: track 82.1 -> 106.5 mm
- net EPD_DC: track 111.0 -> 87.0 mm, vias 4 -> 2
- net VBAT: track 176.5 -> 156.5 mm, vias 6 -> 5
- net VBUS: track 201.7 -> 183.8 mm, vias 6 -> 2
- net GND: track 723.0 -> 705.6 mm, vias 11 -> 15
- net RX: track 40.1 -> 22.9 mm, vias 0 -> 2
- net INT_RTC: track 119.5 -> 103.0 mm, vias 0 -> 5
- net SCL: track 196.9 -> 210.8 mm
- net SDA: track 200.7 -> 186.9 mm, vias 6 -> 7
- net SS_SD: track 170.7 -> 183.8 mm, vias 5 -> 2
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Other:
- outline, holes or cut-outs redrawn
