File: Hardware/E-book_Reader.sch (EAGLE design)
At the start: 103 parts, among them IC1 BD5229G-TR, IC4 XC6220A331MR-G, J1 FH34SRJ-24S-0.5SH_99_, J2 SAMACSYS_PARTS_USB4110-GF-A, J3 QWIIC_RIGHT_ANGLE, J4 112A-TAAR-R03_ATTEND, Q1 20V/4.2A/52mΩ/1.4W, Q2 20V/4.2A/52mΩ/1.4W, Q3 SI1308EDL-T1-GE3, U1 W25Q512JVEIQ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

Commit message: Add files via upload
Parts:
- removed R2_PINH5: 10k, DeskAssistant v19 v1:ESP32_WROVER_EAGLE-LTSPICE_RR0402
- added R1: 10k, DeskAssistant v19 v1:ESP32_WROVER_EAGLE-LTSPICE_RR0402
Connections:
- net 3V3: now also R1.1, R5.2; no longer R2_PINH5.2, R5.1
- net FLASH_CS: now also R5.1; no longer R2_PINH5.1
- net GPIO8: now also R1.2; no longer R5.2
Other:
- note added: "69"
- moved on the sheet: R5
